File: main v0.04.sch (EAGLE design)
At the start: 66 parts, among them IC1 4050D, U1 MCP73831, U2 TPS61200, U3 MAX1704X, U4 USD-SOCKETNEW, X1 USB-MICROB, Y1 16MHz KX-7

Commit message: Clean up of schematics
General clean up + 5V reg added + On/off control connected
Parts:
- removed SJ2: UVLO Disable, SparkFun-Passives:SOLDERJUMPERNO
- added C22: 22uF, SparkFun:CAP0805
- added C23, C24: 0.1uF, SparkFun:CAP0805
- added C25: 10uF, SparkFun:CAP0805
- added L3: 4.7uH, 1.2A, SparkFun:INDUCTOR.
- added R20: 2M, SparkFun:RESISTOR0805-RES
- added R21: 220k, SparkFun:RESISTOR0805-RES
- added U5: TPS61200, SparkFun:TPS61200
- R11: value 10k -> 2M
- R12: value 10k -> 220k
- renumbered HMC8339 to HMC5883, U$2 to FER
Connections:
- removed net EN: R11.2, U2.EN
- removed net N$22: C21.2, Q1PMOS.S, R19.2
- removed net PS: R12.2, U2.PS
- removed net VBAT: C20.2, Q1PMOS.D, R16.2, R17.2
- removed net VBATT: C10.1, C11.1, C16.1, JP2.2, L2.2, R11.1, R12.1, R3.2, SJ2.2, U1.VBAT, U2.VIN
- new net 5V: C22.1, R20.2, U5.VOUT
- new net EN5V: U5.EN
- new net N$16: L3.1, U5.L
- new net N$17: C24.1, U5.VAUX
- new net UVLO1: C23.2, R11.1, R12.2, U5.UVLO
- new net VIN: C11.1, C16.1, C21.2, C23.1, C25.1, L2.2, L3.2, Q1PMOS.S, R11.2, R19.2, R3.2, U2.EN, U2.PS, U2.VIN, U5.PS, U5.VIN
- new net V_BATT: C10.1, C20.2, JP2.2, Q1PMOS.D, R14.2, R15.2, R16.2, R17.2, U1.VBAT
- net AUX_SCL: now also HMC5883.4
- net AUX_SDA: now also HMC5883.3
- net FB: now also R20.1, R21.2, U5.FB
- net GND: now also C22.2, C24.2, C25.2, U5.PAD@1, U5.PAD@2, U5.PAD@3, U5.PAD@4, U5.PAD@5, U5.PGND
- net GND1: now also R12.1, R21.1, U5.GND
- net SCL: no longer HMC5883.4
- net SDA: no longer HMC5883.3
- net UVLO: no longer SJ2.1
- net VCC: no longer R14.2, R15.2
Other:
- note added: "Battery Level Measurement"
- note added: "Sensors"
- note added: "Switching Regulator 3.3V"
- note added: "Switching Regulator 5V"
- note added: "Turn on/off control"
- note added: "µC"
- note added: "µSD Card"
- note removed: "*close jumper SJ2 to disable UVLO*"
- note removed: "Switching Regulator"
- moved on the sheet: ATMEGA, C1, C11, C15, C16, C19, C2, C20, C3, C4, C5, C6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
